File: RPC-PC-hardware/RPC-PC-hardware.kicad_pcb (KiCad board)
At the start: 2 copper layers, 46 x 38 mm, 46 parts, among them J1 USB_C_Receptacle_USB2.0_16P, J3 Conn_02x05_Odd_Even, J4 Conn_02x05_Odd_Even, J5 Conn_01x03, SW3 SW_Push, SW4 SW_Push, SW5 SW_Push, U1 ESP32-C3-WROOM-02, U2 TCMT1100, U3 BQ25186DLHR, U5 TCMT1100, U6 DS8572-33S5, U8 TCMT1100, U9 SK12D07VG4

Commit message: added production files
Parts:
- added REF**: MONKE, 1_RPC_PC:Untitled, B.Cu at (0.00, 0.00)
Other:
- board text added: "Abdelrahman Elbarkouky 13/10/2026"
